Commit message: grasping solved

File: panda_description/urdf/gazebo.xacro (robot description, xacro)
@@ -3,17 +3,7 @@
   <xacro:property name="PI" value="3.14159265359" />
   <ros2_control name="RobotSystem" type="system">
-    <!-- ros2_control Gazebo -->
-    <!-- ROS 2 Humble -->
-    <xacro:if value="$(arg is_ignition)">
-      <hardware>
-        <plugin>ign_ros2_control/IgnitionSystem</plugin>
-      </hardware>
-    </xacro:if>
-    <!-- ROS 2 Iron or above -->
-    <xacro:unless value="$(arg is_ignition)">
-      <hardware>
-        <plugin>gz_ros2_control/GazeboSimSystem</plugin>
-      </hardware>
-    </xacro:unless>
+    <hardware>
+      <plugin>gz_ros2_control/GazeboSimSystem</plugin>
+    </hardware>
     <!-- Joint 1 -->
     <joint name="panda_joint1">
@@ -46,5 +36,7 @@
         <param name="max">0.0</param>
       </command_interface>
-      <state_interface name="position"/>
+      <state_interface name="position">
+        <param name="initial_value">-0.1</param>
+      </state_interface>
     </joint>
     <!-- Joint 5 -->

File: panda_description/urdf/ros2control.xacro (robot description, xacro)
@@ -2,19 +2,47 @@
 <robot xmlns:xacro="http://www.ros.org/wiki/xacro" name="panda">
   <!-- ROS 2 Control -->
-  <!-- ROS 2 Humble -->
   <gazebo>
+    <plugin filename="gz_ros2_control-system" name="gz_ros2_control::GazeboSimROS2ControlPlugin">
+      <parameters>$(find panda_controller)/config/controllers.yaml</parameters>
+    </plugin>
+    <!--
+      SDFormat collapses the fixed panda_hand joint into panda_link7, so
+      detachable joints must use panda_link7 as the parent link entity.
+    -->
+    <plugin filename="ignition-gazebo-detachable-joint-system"
+            name="ignition::gazebo::systems::DetachableJoint">
+      <parent_link>panda_link7</parent_link>
+      <child_model>red_box</child_model>
+      <child_link>red_link</child_link>
+      <detach_topic>/panda_pick/red/detach</detach_topic>
+      <attach_topic>/panda_pick/red/attach</attach_topic>
+      <output_topic>/panda_pick/red/state</output_topic>
+    </plugin>
+    <plugin filename="ignition-gazebo-detachable-joint-system"
+            name="ignition::gazebo::systems::DetachableJoint">
+      <parent_link>panda_link7</parent_link>
+      <child_model>green_box</child_model>
+      <child_link>green_link</child_link>
+      <detach_topic>/panda_pick/green/detach</detach_topic>
+      <attach_topic>/panda_pick/green/attach</attach_topic>
+      <output_topic>/panda_pick/green/state</output_topic>
+    </plugin>
+    <plugin filename="ignition-gazebo-detachable-joint-system"
+            name="ignition::gazebo::systems::DetachableJoint">
+      <parent_link>panda_link7</parent_link>
+      <child_model>blue_box</child_model>
+      <child_link>blue_link</child_link>
+      <detach_topic>/panda_pick/blue/detach</detach_topic>
+      <attach_topic>/panda_pick/blue/attach</attach_topic>
+      <output_topic>/panda_pick/blue/state</output_topic>
+    </plugin>
+    <!-- ROS 2 Humble / Ignition Gazebo -->
     <xacro:if value="$(arg is_ignition)">
-      <plugin filename="ign_ros2_control-system" name="ign_ros2_control::IgnitionROS2ControlPlugin">
-        <parameters>$(find panda_controller)/config/controllers.yaml</parameters>
-      </plugin>
       <plugin filename="ignition-gazebo-sensors-system" name="ignition::gazebo::systems::Sensors">
         <render_engine>ogre2</render_engine>
       </plugin>
     </xacro:if>
-    <!-- ROS 2 Iron or above -->
+    <!-- ROS 2 Iron or newer / Gazebo -->
     <xacro:unless value="$(arg is_ignition)">
-      <plugin filename="gz_ros2_control-system" name="gz_ros2_control::GazeboSimROS2ControlPlugin">
-        <parameters>$(find panda_controller)/config/controllers.yaml</parameters>
-      </plugin>
       <plugin filename="gz-sim-sensors-system" name="gz::sim::systems::Sensors">
         <render_engine>ogre2</render_engine>

File: panda_description/urdf/sensors.xacro (robot description, xacro)
@@ -12,5 +12,7 @@
                 <box size="0.1 0.1 0.05"/>
             </geometry>
-            <material name="red"/>
+            <material name="camera_red">
+                <color rgba="0.8 0.0 0.0 1.0"/>
+            </material>
         </visual>
         <collision>
@@ -19,5 +21,4 @@
                 <box size="0.1 0.1 0.05"/>
             </geometry>
-            <material name="red"/>
         </collision>
     </link>
@@ -35,5 +36,5 @@
     <gazebo reference="camera_link">
         <sensor name="camera" type="camera">
-            <pose>0 0 0 0 1.57 0</pose>
+            <pose>0 0 0 0 ${pi/2} 0</pose>
             <visualize>true</visualize>
             <update_rate>10.0</update_rate>
